Commit message: Depth works

File: urdf/turtlebot3_waffle.urdf (robot description, URDF)
Before this commit: robot turtlebot3_waffle, 13 links, 12 joints
Joints:
- joint camera_depth_joint: origin xyz=0.005 0.028 0.013 rpy=0 0 0 -> xyz=0.005 0.018 0.033 rpy=0 0 0

Commit message: Changing depth camera position

File: urdf/turtlebot3_waffle.urdf (robot description, URDF)
Before this commit: robot turtlebot3_waffle, 13 links, 12 joints
Joints:
- joint camera_depth_joint: origin xyz=0.005 0.018 0.033 rpy=0 0 0 -> xyz=0.005 0.018 0.013 rpy=0 0 0
